Commit message: fix(web): position joint 5 at wrist center and fix http response order

File: src/yaskawa_workcell_description/urdf/gp8_macro.xacro (robot description, xacro)
@@ -127,5 +127,5 @@
       <parent link="${prefix}link_4_r"/>
       <child link="${prefix}link_5_b"/>
-      <origin xyz="0.15 0 0" rpy="0 0 0"/>
+      <origin xyz="0 0 0" rpy="0 0 0"/>
       <axis xyz="0 1 0"/>
       <limit lower="-2.356" upper="2.356" effort="50.0" velocity="9.60"/>
